File: _autosave-prototype-physical modular.kicad_pcb (KiCad board)
At the start: 2 copper layers, 100 x 164 mm, 177 parts, among them CON1 BARREL_JACK, CON2 SD_Card, IC1 ATMEGA2560-A, J1 MIDI_IN, J2 MIDI_OUT, P1 POWER, P13 PD, P15 PH, P16 PF, P17 SD_PINS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

Commit message: update gerbers
Parts:
- added >NAME: >VALUE, SeeedOPL-Connector:AUDIO6P-SMD-3.5-14.0X6.4X5.0MM, F.Cu at (106.8, -7.30)
- added >NAME: >VALUE, SeeedOPL-Connector:AUDIO6P-SMD-3.5-14.0X6.4X5.0MM, F.Cu at (55.5, -32.3)
Other:
- board text added: "add more copper to power dissipation of power regulators"
